File: usb-breadboard-power.kicad_sch (KiCad schematic)
At the start: 54 parts, among them J1 USB_C_Receptacle_PowerOnly_6P, J2 Conn_01x03, J3 Conn_02x02, J4 Conn_02x02, Q1 Q_PMOS_GSD, Q2 Q_PMOS_GSD, SW1 SW_DIP_x03, U1 CYPD3177, U2 LM339, U3 AP63203WU

Commit message: Added jumper shunts to BOM
Parts:
- added JS1, JS2: ~, symbol usb-breadboard:jumper-shunt
- JP1, JP2: now in the parts list
Connections:
- net at U1.17 (VBUS_IN): now also C1.1, C2.1, F1.2, Q1.3 (D), R1.1
Other:
- note added: "Shunts for jumpers for the BOM"
Changed lines of the file:
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@@
     (fill (type none))
   )
-  (rectangle (start 177.8 104.14) (end 238.76 160.02)
+  (rectangle (start 177.8 104.14) (end 252.73 160.02)
     (stroke (width 0) (type default))
     (fill (type none))
@@
   (text "3.3v Regulator" (at 88.9 139.7 0)
     (effects (font (size 2.5 2.5)) (justify left bottom))
+  )
+  (text "Shunts for jumpers\nfor the BOM" (at 231.14 155.575 0)
+    (effects (font (size 1.27 1.27)) (justify left bottom))
   )
   (text "3v3" (at 165.1 157.48 0)
@@
     )
   )
+  (symbol (lib_id "usb-breadboard:jumper-shunt") (at 243.205 144.78 0) (unit 1)
+    (in_bom yes) (on_board no) (dnp no) (fields_autoplaced)
+    (property "Reference" "JS2" (at 245.745 148.59 0)
+      (effects (font (size 1.27 1.27)) (justify left))
+    )
+    (property "Value" "~" (at 243.205 144.78 0)
+      (effects (font (size 1.27 1.27)))
+    )
+    (property "Footprint" "" (at 243.205 144.78 0)
+      (effects (font (size 1.27 1.27)) hide)
+    )
+    (property "Datasheet" "" (at 243.205 144.78 0)
+      (effects (font (size 1.27 1.27)) hide)
+    )
+    (property "DPN-m" "855-M7581-05" (at 243.205 144.78 0)
+      (effects (font (size 1.27 1.27)) hide)
+    )
+    (property "MPN-m" "M7581-05" (at 243.205 144.78 0)
+      (effects (font (size 1.27 1.27)) hide)
+    )
+    (instances
+      (project "usb-breadboard-power"
+        (path "/e7c97585-576c-43b2-a997-16cefae3bf47"
+          (reference "JS2") (unit 1)
+        )
+      )
+    )
+  )
   (symbol (lib_id "power:GND") (at 241.3 30.48 0) (unit 1)
     (in_bom yes) (on_board yes) (dnp no) (fields_autoplaced)
@@
   )
   (symbol (lib_id "Jumper:Jumper_3_Bridged12") (at 195.58 121.92 0) (mirror y) (unit 1)
-    (in_bom no) (on_board yes) (dnp no)
+    (in_bom yes) (on_board yes) (dnp no)
     (property "Reference" "JP1" (at 195.58 116.84 0)
       (effects (font (size 1.27 1.27)))
@@
     )
   )
+  (symbol (lib_id "usb-breadboard:jumper-shunt") (at 233.68 144.78 0) (unit 1)
+    (in_bom yes) (on_board no) (dnp no) (fields_autoplaced)
+    (property "Reference" "JS1" (at 236.22 148.59 0)
+      (effects (font (size 1.27 1.27)) (justify left))
+    )
+    (property "Value" "~" (at 233.68 144.78 0)
+      (effects (font (size 1.27 1.27)))
+    )
+    (property "Footprint" "" (at 233.68 144.78 0)
+      (effects (font (size 1.27 1.27)) hide)
+    )
+    (property "Datasheet" "" (at 233.68 144.78 0)
+      (effects (font (size 1.27 1.27)) hide)
+    )
+    (property "DPN-m" "855-M7581-05" (at 233.68 144.78 0)
+      (effects (font (size 1.27 1.27)) hide)
+    )
+    (property "MPN-m" "M7581-05" (at 233.68 144.78 0)
+      (effects (font (size 1.27 1.27)) hide)
+    )
+    (instances
+      (project "usb-breadboard-power"
+        (path "/e7c97585-576c-43b2-a997-16cefae3bf47"
+          (reference "JS1") (unit 1)
+        )
+      )
+    )
+  )
   (symbol (lib_id "Device:R") (at 111.76 85.09 0) (mirror y) (unit 1)
     (in_bom yes) (on_board yes) (dnp no) (fields_autoplaced)
@@
   )
   (symbol (lib_id "Jumper:Jumper_3_Bridged12") (at 223.52 121.92 0) (mirror y) (unit 1)
-    (in_bom no) (on_board yes) (dnp no)
+    (in_bom yes) (on_board yes) (dnp no)
     (property "Reference" "JP2" (at 223.52 116.84 0)
       (effects (font (size 1.27 1.27)))

Commit message: Fixed issues discovered while building first run
Parts:
- J2: value Conn_01x03 -> DNP
- RN1, RN2: footprint Resistor_SMD:R_Array_Convex_4x1206 -> usb-breadboard:CAY16472J4LF
Connections:
- net at C1.1, C2.1, F1.2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: now also U1.18 (VBUS_IN); no longer U1.17 (VBUS_IN)
Changed lines of the file:
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@@
       (effects (font (size 1.27 1.27)) (justify left))
     )
-    (property "Value" "Conn_01x03" (at 106.68 67.945 0)
+    (property "Value" "DNP" (at 106.68 67.945 0)
       (effects (font (size 1.27 1.27)) (justify left))
     )
@@
     (pin "16")
     (pin "17")
-    (pin "17")
+    (pin "18")
     (pin "19")
     (pin "2")
@@
       (effects (font (size 1.27 1.27)) (justify right))
     )
-    (property "Footprint" "Resistor_SMD:R_Array_Convex_4x1206" (at 200.66 65.405 90)
+    (property "Footprint" "usb-breadboard:CAY16472J4LF" (at 200.66 65.405 90)
       (effects (font (size 1.27 1.27)) hide)
     )
@@
       (effects (font (size 1.27 1.27)))
     )
-    (property "Footprint" "Resistor_SMD:R_Array_Convex_4x1206" (at 269.24 51.435 90)
-      (effects (font (size 1.27 1.27)) hide)
-    )
+    (property "Footprint" "usb-breadboard:CAY16472J4LF" (at 269.24 51.435 90)
+      (effects (font (size 1.27 1.27)) hide)
+    )
