File: usb-breadboard-power.kicad_pcb (KiCad board)
At the start: 2 copper layers, 53 x 25.7 mm, 54 parts, among them J1 USB_C_Receptacle_PowerOnly_6P, J2 DNP, J3 Conn_02x02, J4 Conn_02x02, Q1 Q_PMOS_GSD, Q2 Q_PMOS_GSD, SW1 SW_DIP_x03, U1 CYPD3177, U2 LM339, U3 AP63203WU

Commit message: Updated documentation
Other:
- board text added: "A"
- board text added: "B"
Changed lines of the file:
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@@
       (drillshape 0)
       (scaleselection 1)
-      (outputdirectory "/media/benjamin/BEN_LAB_USB/bbps-test1-osh/")
+      (outputdirectory "./board")
     )
   )
@@
     (effects (font (size 0.8 0.8) (thickness 0.12)) (justify left bottom))
   )
+  (gr_text "B" (at 109.15 99.35) (layer "F.SilkS")
+    (effects (font (size 1 1) (thickness 0.15)) (justify left bottom))
+  )
   (gr_text "20" (at 122.5 95.9) (layer "F.SilkS")
     (effects (font (size 1 1) (thickness 0.15)) (justify left bottom))
@@
     (effects (font (size 1 1) (thickness 0.15)) (justify left bottom))
   )
+  (gr_text "A" (at 109.15 108.5) (layer "F.SilkS")
+    (effects (font (size 1 1) (thickness 0.15)) (justify left bottom))
+  )

Commit message: Added info to back of board
Other:
- board text added: "12V*"
- board text added: "15V"
- board text added: "20V"
- board text added: "5V"
- board text added: "9V"
- board text added: "S1"
- board text added: "S2"
- board text added: "S3"
- board text added: "USBC Breadboard Power Supply V1.0"
- board text added: "VBus Selection"
- board text added: "https://github.com/Benjamin-C/USB-C-BBPS"
- board text added: "x"
- board text removed: "V1.0"
